File: MainPCB.sch (EAGLE design)
At the start: 13 parts, among them J2 DCJ0202

Commit message: fixin the things
Parts:
- removed U$2: MFRC522, SeniorDesignParts:MFRC522
- added JP1: (no value), pinhead:PINHD-2X6
Connections:
- removed net SID: J1.14
- new net MISO: JP1.5, U$1.PC2
- new net MOSI: J1.14, JP1.2, U$1.PB15
- new net SS: JP1.10, U$1.PC6
- net +5V: no longer J1.3
- net 3.3V: now also JP1.1
- net CSB: now also U$1.PC9
- net GND: now also J1.3, JP1.11; no longer U$2.GND
- net RS: now also U$1.PC8
- net SCLK: now also JP1.6, U$1.PB13
Other:
- note added: "POWER"
Changed lines of the file:
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@@
 <part name="P+1" library="supply1" library_urn="urn:adsk.eagle:library:371" deviceset="+5V" device=""/>
 <part name="GND2" library="supply1" library_urn="urn:adsk.eagle:library:371" deviceset="GND" device=""/>
-<part name="U$2" library="SeniorDesignParts" deviceset="MFRC522" device=""/>
 <part name="FRAME1" library="frames" library_urn="urn:adsk.eagle:library:229" deviceset="A4L-LOC" device=""/>
 <part name="FRAME2" library="frames" library_urn="urn:adsk.eagle:library:229" deviceset="A4L-LOC" device=""/>
@@
 <part name="P+3" library="supply1" library_urn="urn:adsk.eagle:library:371" deviceset="+5V" device=""/>
 <part name="GND6" library="SparkFun-PowerSymbols" library_urn="urn:adsk.eagle:library:530" deviceset="GND" device=""/>
-<part name="GND7" library="SparkFun-PowerSymbols" library_urn="urn:adsk.eagle:library:530" deviceset="GND" device=""/>
 <part name="J2" library="con-jack" library_urn="urn:adsk.eagle:library:154" deviceset="DCJ0202" device="" package3d_urn="urn:adsk.eagle:package:7491/1"/>
 <part name="GND8" library="SparkFun-PowerSymbols" library_urn="urn:adsk.eagle:library:530" deviceset="GND" device=""/>
@@
 <part name="GND11" library="supply1" library_urn="urn:adsk.eagle:library:371" deviceset="GND" device=""/>
 <part name="SUPPLY3" library="SparkFun-PowerSymbols" library_urn="urn:adsk.eagle:library:530" deviceset="3.3V" device=""/>
+<part name="JP1" library="pinhead" library_urn="urn:adsk.eagle:library:325" deviceset="PINHD-2X6" device="" package3d_urn="urn:adsk.eagle:package:22474/2"/>
+<part name="SUPPLY4" library="SparkFun-PowerSymbols" library_urn="urn:adsk.eagle:library:530" deviceset="3.3V" device=""/>
+<part name="GND12" library="supply1" library_urn="urn:adsk.eagle:library:371" deviceset="GND" device=""/>
 </parts>
 <sheets>
@@
 <text x="162.56" y="12.7" size="3.81" layer="95">STM32F0 Connections</text>
 <text x="289.56" y="157.48" size="3.81" layer="95">LCD Connections</text>
+<text x="35.56" y="347.98" size="3.81" layer="97">POWER</text>
 </plain>
 <instances>
@@
 <attribute name="VALUE" x="330.2" y="93.98" size="1.778" layer="96"/>
 </instance>
-<instance part="P+1" gate="1" x="342.9" y="119.38">
-<attribute name="VALUE" x="340.36" y="114.3" size="1.778" layer="96" rot="R90"/>
+<instance part="P+1" gate="1" x="342.9" y="116.84">
+<attribute name="VALUE" x="340.36" y="111.76" size="1.778" layer="96" rot="R90"/>
 </instance>
 <instance part="GND2" gate="1" x="307.34" y="147.32">
 <attribute name="VALUE" x="304.8" y="144.78" size="1.778" layer="96"/>
 </instance>
-<instance part="U$2" gate="G$1" x="403.86" y="299.72"/>
 <instance part="FRAME1" gate="G$1" x="0" y="0">
 <attribute name="DRAWING_NAME" x="217.17" y="15.24" size="2.54" layer="94"/>
@@
 <instance part="GND6" gate="1" x="76.2" y="299.72">
 <attribute name="VALUE" x="76.2" y="299.466" size="1.778" layer="96" align="top-center"/>
-</instance>
-<instance part="GND7" gate="1" x="411.48" y="238.76">
-<attribute name="VALUE" x="411.48" y="238.506" size="1.778" layer="96" align="top-center"/>
 </instance>
 <instance part="J2" gate="G$1" x="27.94" y="264.16">
@@
 <attribute name="VALUE" x="403.86" y="150.114" size="1.778" layer="96" align="bottom-center"/>
 </instance>
+<instance part="JP1" gate="A" x="312.42" y="317.5">
+<attribute name="NAME" x="306.07" y="325.755" size="1.778" layer="95"/>
+<attribute name="VALUE" x="306.07" y="304.8" size="1.778" layer="96"/>
+</instance>
+<instance part="SUPPLY4" gate="G$1" x="297.18" y="332.74">
+<attribute name="VALUE" x="297.18" y="335.534" size="1.778" layer="96" align="bottom-center"/>
+</instance>
+<instance part="GND12" gate="1" x="297.18" y="299.72">
+<attribute name="VALUE" x="294.64" y="297.18" size="1.778" layer="96"/>
+</instance>
 </instances>
 <busses>
@@
 <wire x1="332.74" y1="106.68" x2="332.74" y2="99.06" width="0.1524" layer="91"/>
 <pinref part="GND1" gate="1" pin="GND"/>
+<pinref part="J1" gate="G$1" pin="3"/>
+<wire x1="325.12" y1="111.76" x2="332.74" y2="111.76" width="0.1524" layer="91"/>
+<wire x1="332.74" y1="111.76" x2="332.74" y2="106.68" width="0.1524" layer="91"/>
+<junction x="332.74" y="106.68"/>
 </segment>
 <segment>
@@
 <wire x1="307.34" y1="152.4" x2="307.34" y2="149.86" width="0.1524" layer="91"/>
 <pinref part="GND2" gate="1" pin="GND"/>
+<label x="312.42" y="152.4" size="1.778" layer="95"/>
 </segment>
 <segment>
@@
 </segment>
 <segment>
-<pinref part="U$2" gate="G$1" pin="GND"/>
-<pinref part="GND7" gate="1" pin="GND"/>
-<wire x1="411.48" y1="248.92" x2="411.48" y2="241.3" width="0.1524" layer="91"/>
-</segment>
-<segment>
 <pinref part="J2" gate="G$1" pin="2"/>
 <pinref part="GND8" gate="1" pin="GND"/>
@@
 <wire x1="434.34" y1="101.6" x2="434.34" y2="93.98" width="0.1524" layer="91"/>
 </segment>
+<segment>
+<pinref part="JP1" gate="A" pin="11"/>
+<wire x1="309.88" y1="309.88" x2="297.18" y2="309.88" width="0.1524" layer="91"/>
+<wire x1="297.18" y1="309.88" x2="297.18" y2="302.26" width="0.1524" layer="91"/>
+<pinref part="GND12" gate="1" pin="GND"/>
+</segment>
 </net>
 <net name="+5V" class="0">
 <segment>
 <pinref part="J1" gate="G$1" pin="2"/>
-<wire x1="325.12" y1="109.22" x2="327.66" y2="109.22" width="0.1524" layer="91"/>
-<wire x1="327.66" y1="109.22" x2="342.9" y2="109.22" width="0.1524" layer="91"/>
-<wire x1="342.9" y1="109.22" x2="342.9" y2="116.84" width="0.1524" layer="91"/>
+<wire x1="325.12" y1="109.22" x2="342.9" y2="109.22" width="0.1524" layer="91"/>
+<wire x1="342.9" y1="109.22" x2="342.9" y2="114.3" width="0.1524" layer="91"/>
 <pinref part="P+1" gate="1" pin="+5V"/>
-<pinref part="J1" gate="G$1" pin="3"/>
-<wire x1="325.12" y1="111.76" x2="327.66" y2="111.76" width="0.1524" layer="91"/>
-<wire x1="327.66" y1="111.76" x2="327.66" y2="109.22" width="0.1524" layer="91"/>
-<junction x="327.66" y="109.22"/>
 </segment>
 <segment>
@@
 <label x="330.2" y="114.3" size="1.778" layer="95"/>
 </segment>
+<segment>
+<pinref part="U$1" gate="G$1" pin="PC8"/>
+<wire x1="116.84" y1="43.18" x2="132.08" y2="43.18" width="0.1524" layer="91"/>
+<label x="127" y="43.18" size="1.778" layer="95"/>
+</segment>
 </net>
 <net name="CSB" class="0">
@@
 <label x="330.2" y="134.62" size="1.778" layer="95"/>
 </segment>
+<segment>
+<pinref part="U$1" gate="G$1" pin="PC9"/>
+<wire x1="116.84" y1="48.26" x2="132.08" y2="48.26" width="0.1524" layer="91"/>
+<label x="127" y="48.26" size="1.778" layer="95"/>
+</segment>
 </net>
 <net name="SCLK" class="0">
@@
 <label x="327.66" y="137.16" size="1.778" layer="95"/>
 </segment>
-</net>
-<net name="SID" class="0">
+<segment>
+<pinref part="U$1" gate="G$1" pin="PB13"/>
+<wire x1="116.84" y1="17.78" x2="132.08" y2="17.78" width="0.1524" layer="91"/>
+<label x="124.46" y="17.78" size="1.778" layer="95"/>
+</segment>
+<segment>
+<pinref part="JP1" gate="A" pin="6"/>
+<wire x1="317.5" y1="317.5" x2="337.82" y2="317.5" width="0.1524" layer="91"/>
+<label x="330.2" y="317.5" size="1.778" layer="95"/>
+</segment>
+</net>
+<net name="MOSI" class="0">
 <segment>
 <pinref part="J1" gate="G$1" pin="14"/>
 <wire x1="325.12" y1="139.7" x2="335.28" y2="139.7" width="0.1524" layer="91"/>
 <label x="330.2" y="139.7" size="1.778" layer="95"/>
+</segment>
+<segment>
+<pinref part="U$1" gate="G$1" pin="PB15"/>
+<wire x1="116.84" y1="27.94" x2="132.08" y2="27.94" width="0.1524" layer="91"/>
+<label x="124.46" y="27.94" size="1.778" layer="95"/>
+</segment>
+<segment>
+<pinref part="JP1" gate="A" pin="2"/>
+<wire x1="317.5" y1="322.58" x2="337.82" y2="322.58" width="0.1524" layer="91"/>
+<label x="330.2" y="322.58" size="1.778" layer="95"/>
 </segment>
 </net>
@@
 <wire x1="403.86" y1="139.7" x2="403.86" y2="147.32" width="0.1524" layer="91"/>
 <pinref part="SUPPLY3" gate="G$1" pin="3.3V"/>
+</segment>
+<segment>
+<pinref part="JP1" gate="A" pin="1"/>
+<wire x1="309.88" y1="322.58" x2="297.18" y2="322.58" width="0.1524" layer="91"/>
+<wire x1="297.18" y1="322.58" x2="297.18" y2="332.74" width="0.1524" layer="91"/>
+<pinref part="SUPPLY4" gate="G$1" pin="3.3V"/>
 </segment>
 </net>
@@
 </segment>
 </net>
+<net name="MISO" class="0">
+<segment>
+<pinref part="JP1" gate="A" pin="5"/>
+<wire x1="309.88" y1="317.5" x2="289.56" y2="317.5" width="0.1524" layer="91"/>
+<label x="292.1" y="317.5" size="1.778" layer="95"/>
+</segment>
+<segment>
+<pinref part="U$1" gate="G$1" pin="PC2"/>
+<wire x1="50.8" y1="124.46" x2="35.56" y2="124.46" width="0.1524" layer="91"/>
+<label x="38.1" y="124.46" size="1.778" layer="95"/>
+</segment>
+</net>
+<net name="SS" class="0">
+<segment>
+<pinref part="JP1" gate="A" pin="10"/>
+<wire x1="317.5" y1="312.42" x2="337.82" y2="312.42" width="0.1524" layer="91"/>
+<label x="332.74" y="312.42" size="1.778" layer="95"/>
+</segment>
+<segment>
+<pinref part="U$1" gate="G$1" pin="PC6"/>
+<wire x1="116.84" y1="33.02" x2="132.08" y2="33.02" width="0.1524" layer="91"/>
+<label x="127" y="33.02" size="1.778" layer="95"/>
+</segment>
+</net>

Commit message: added bypass capcitors
Parts:
- added C10, C11, C5, C6, C7, C8, C9: 0.1uF, SparkFun-Capacitors:0.1UF-0603-100V-10%
- added JP2: PINHD-1X6, audio amplifier example:PINHD-1X6
- added JP3: (no value), pinhead:PINHD-2X9
Connections:
- new net NRST: JP2.5, U$1.NRST
- new net RX_ESP: U$1.PB6, U$7.RXD0
- new net SWDIO: JP2.4, U$1.PA13
- new net SWO: JP2.6, U$1.PB3
- new net SW_CLK: JP2.2, U$1.PA14
- new net TX_ESP: U$1.PB7, U$7.TXD0
- net +5V: now also C9.1
- net 3.3V: now also C10.1, C11.1, C5.1, C6.1, C7.1, C8.1, JP2.1, U$1.VDD, U$1.VDDA/VREF+, U$1.VDD_1, U$1.VDD_2, U$1.VDD_3
- net GND: now also C10.2, C11.2, C5.2, C6.2, C7.2, C8.2, C9.2, JP2.3, U$1.VSS, U$1.VSSA/VREF-, U$1.VSS_1, U$1.VSS_2, U$1.VSS_3

Commit message: added various parts
Parts:
- removed JP3: (no value), pinhead:PINHD-2X9
- added H1, H2, H3, H4: STAND-OFF, SparkFun-Hardware:STAND-OFF
- added JP5: (no value), pinhead:PINHD-1X18
- added R1, R2, R3, R4, R5, R6, R7, R8, R9: 1k, SparkFun-Resistors:1KOHM-0603-1/10W-1%
- added U$10, U$2, U$9: TSV914AIDT, SeniorDesignParts:TSV914AIDT
Connections:
- new net ROW1: JP5.1, R3.1, U$2.1IN-
- new net ROW2: JP5.2, R2.1, U$2.2IN-
- new net ROW3: JP5.3, R1.1, U$2.3IN-
- new net ROW4: JP5.4, R6.1, U$9.1IN-
- new net ROW5: JP5.5, R5.1, U$9.2IN-
- new net ROW6: JP5.6, R4.1, U$9.3IN-
- new net ROW7: JP5.7, R9.1, U$10.1IN-
- new net ROW8: JP5.8, R8.1, U$10.2IN-
- new net ROW9: JP5.9, R7.1, U$10.3IN-
- new net ROWOUT_1: R3.2, U$1.PA1, U$2.1OUT
- new net ROWOUT_2: R2.2, U$1.PA2, U$2.2OUT
- new net ROWOUT_3: R1.2, U$1.PA3, U$2.3OUT
- new net ROWOUT_4: R6.2, U$1.PA4, U$9.1OUT
- new net ROWOUT_5: R5.2, U$1.PA5, U$9.2OUT
- new net ROWOUT_6: R4.2, U$1.PA6, U$9.3OUT
- new net ROWOUT_7: R9.2, U$1.PA7, U$10.1OUT
- new net ROWOUT_8: R8.2, U$1.PB0, U$10.2OUT
- new net ROWOUT_9: R7.2, U$1.PB1, U$10.3OUT
- net +5V: now also U$10.VCC+, U$2.VCC+, U$9.VCC+
- net GND: now also U$10.1IN+, U$10.2IN+, U$10.3IN+, U$10.GND, U$2.1IN+, U$2.2IN+, U$2.3IN+, U$2.GND, U$9.1IN+, U$9.2IN+, U$9.3IN+, U$9.GND
Other:
- moved on the sheet: JP1
