File: MainPCB.brd (EAGLE design)
At the start: 139.7 x 76.2 mm, 71 parts, among them J2 DCJ0202, J3 FEMALE 2x3, X1 8MHz

Commit message: yay purty
Parts:
- removed H1, H5: STAND-OFF, SparkFun-Hardware:STAND-OFF
- moved C24 81.6 mm to (12.9, 47.5), flipped to the bottom, turned to 180 degrees
- moved C11 81.1 mm to (11.6, 53.2), flipped to the bottom, turned to 90 degrees
- moved U1 70.3 mm to (5.54, 51.5), flipped to the bottom, turned to 270 degrees
- moved R14 11.1 mm to (128.4, 50.7)
- moved U$12 10.6 mm to (124.5, 16.5)
- moved D2 10.3 mm to (120.1, 64.5), turned to 90 degrees
- moved D1 10.0 mm to (117.3, 64.6), turned to 90 degrees
- moved H2 6.07 mm to (20.9, 69.4)
- moved R11 4.68 mm to (120.0, 60.5), turned to 90 degrees
- moved R15 4.66 mm to (128.3, 47.2)
- moved R10 3.97 mm to (117.3, 60.6), turned to 90 degrees
- moved R13 3.86 mm to (97.4, 61.3), turned to 270 degrees
- moved C14 2.43 mm to (88.8, 70.6), flipped to the top
- moved R16 1.27 mm to (128.3, 43.7)
- moved J4 1.22 mm to (119.0, 71.6)
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Connections:
- removed net SS: U$1.37
- new net EN: J4.3
- new net FB1: U$9.13, U$9.14
- new net FB2: U$2.13, U$2.14
- new net FB3: U$10.13, U$10.14
- new net RST_ESP: J4.5
- net 3.3V: now also J4.7
- net GND: now also J4.2, U$10.12, U$2.12, U$9.12
- net RX_ESP: now also J4.8
- net SDA: now also U$1.37
- net TX_ESP: now also J4.1
Routing:
- net 3.3V: track 219.7 -> 397.9 mm, vias 6 -> 5
- net MOSI: track 3.85 -> 105.5 mm, vias 1 -> 3
- net SDA: track 0.00 -> 97.2 mm, vias 0 -> 1
- net MISO: track 3.87 -> 69.6 mm, vias 0 -> 1
- net ROWOUT_2: track 3.96 -> 68.6 mm, vias 0 -> 1
- net +5V: track 5.04 -> 67.8 mm, vias 0 -> 1
- net RS: track 7.75 -> 69.1 mm, vias 0 -> 1
- net ROWOUT_1: track 12.9 -> 73.9 mm
- net ROWOUT_4: track 18.3 -> 70.6 mm
- net COLOUT_2: track 17.2 -> 66.0 mm
- net SCLK: track 0.05 -> 48.5 mm, vias 0 -> 1
- net ROWOUT_5: track 8.71 -> 55.1 mm
- net COLOUT_1: track 15.2 -> 60.7 mm
- net ROWOUT_7: track 10.9 -> 56.1 mm
- net ROWOUT_3: track 12.4 -> 55.3 mm
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- added copper zone on layer 1, net +5V
- added copper zone on layer 16, net +5V
Other:
- board text added: "+5V"
- board text added: "3V3 CLK GND DIO NRST SWO"
- board text added: "DOWN"
- board text added: "GND"
- board text added: "SELECT"
- board text added: "SWO NRST DIO GND CLK 3V3"
- board text added: "UP"
